Commit message: demo for robot on track

File: data/panda/panda.urdf (robot description, URDF)
Before this commit: robot panda, 12 links, 11 joints
Links:
- added link track_x; visual box size=1 0.1 0.1
- added link track_y; visual box size=0.1 1 0.2
Joints:
- added joint move_x: type prismatic, parent track_x, child track_y, origin xyz=0 0 0 rpy=0 0 0, axis 1 0 0, limit lower=-1 upper=1 effort=20 velocity=0.2
- added joint move_y: type prismatic, parent track_y, child panda_link0, origin xyz=0 0 0 rpy=0 0 0, axis 0 1 0, limit lower=-1 upper=1 effort=20 velocity=0.2
