Commit message: moved up panda so it's not touching the ground

File: data/panda/panda_on_rail.urdf (robot description, URDF)
Before this commit: robot panda, 14 links, 13 joints
Links:
- link track_y: geometry visual box size=0.1 1 0.1
Joints:
- joint move_x: origin xyz=0 0 0 rpy=0 0 0 -> xyz=0 0 0.01 rpy=0 0 0
- joint move_y: origin xyz=0 0 0 rpy=0 0 0 -> xyz=0 0 0.01 rpy=0 0 0
